File: kicad/macropad.kicad_sch (KiCad schematic)
At the start: 15 parts, among them J1 Conn_01x04_Socket, SW1 CherryMX, SW10 RotaryEncoder_Switch, SW11 RotaryEncoder_Switch, SW12 SW_Push, SW2 CherryMX, SW3 CherryMX, SW4 CherryMX, SW5 CherryMX, SW6 CherryMX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

Commit message: updated design
Parts:
- SW10, SW11: footprint Rotary_Encoder:RotaryEncoder_Alps_EC11E-Switch_Vertical_H20mm -> Macropad_Library:RotaryEncoder
- U1: footprint footprints:RPi_Pico_SMD_TH -> Macropad_Library:RPi_Pico_SMD_TH
Changed lines of the file:
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@@
 			)
 		)
-		(property "Footprint" "Rotary_Encoder:RotaryEncoder_Alps_EC11E-Switch_Vertical_H20mm"
+		(property "Footprint" "Macropad_Library:RotaryEncoder"
 			(at 191.77 46.736 0)
 			(effects
@@
 			)
 		)
-		(property "Footprint" "Rotary_Encoder:RotaryEncoder_Alps_EC11E-Switch_Vertical_H20mm"
+		(property "Footprint" "Macropad_Library:RotaryEncoder"
 			(at 198.12 67.056 0)
 			(effects
@@
 		(on_board yes)
 		(dnp no)
-		(fields_autoplaced yes)
 		(property "Reference" "J1"
 			(at 201.295 93.98 0)
@@
 		)
 		(property "Footprint" "Connector_PinHeader_2.54mm:PinHeader_1x04_P2.54mm_Vertical"
-			(at 201.93 83.82 0)
-			(effects
-				(font
-					(size 1.27 1.27)
-				)
-				(hide yes)
+			(at 235.458 82.55 0)
+			(effects
+				(font
+					(size 1.27 1.27)
+				)
 			)
 		)
@@
 			)
 		)
-		(property "Footprint" "footprints:RPi_Pico_SMD_TH"
+		(property "Footprint" "Macropad_Library:RPi_Pico_SMD_TH"
 			(at 153.67 73.66 90)
 			(effects

Commit message: added 3D models
Parts:
- J1: footprint Connector_PinHeader_2.54mm:PinHeader_1x04_P2.54mm_Vertical -> Macropad_Library:SSD1306
- SW1, SW2, SW3, SW4, SW5, SW6, SW7, SW8, SW9: footprint Button_Switch_Keyboard:SW_Cherry_MX_1.00u_PCB -> Macropad_Library:SW_Cherry_MX_1.00u_PCB
- SW12: footprint Button_Switch_THT:SW_PUSH-12mm -> Macropad_Library:SW_PUSH-12mm
Changed lines of the file:
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@@
 			)
 		)
-		(property "Footprint" "Button_Switch_Keyboard:SW_Cherry_MX_1.00u_PCB"
+		(property "Footprint" "Macropad_Library:SW_Cherry_MX_1.00u_PCB"
 			(at 99.06 85.725 0)
 			(effects
@@
 			)
 		)
-		(property "Footprint" "Button_Switch_Keyboard:SW_Cherry_MX_1.00u_PCB"
+		(property "Footprint" "Macropad_Library:SW_Cherry_MX_1.00u_PCB"
 			(at 104.14 121.285 0)
 			(effects
@@
 			)
 		)
-		(property "Footprint" "Button_Switch_Keyboard:SW_Cherry_MX_1.00u_PCB"
+		(property "Footprint" "Macropad_Library:SW_Cherry_MX_1.00u_PCB"
 			(at 104.14 132.715 0)
 			(effects
@@
 			)
 		)
-		(property "Footprint" "Button_Switch_Keyboard:SW_Cherry_MX_1.00u_PCB"
+		(property "Footprint" "Macropad_Library:SW_Cherry_MX_1.00u_PCB"
 			(at 110.49 60.325 0)
 			(effects
@@
 			)
 		)
-		(property "Footprint" "Button_Switch_Keyboard:SW_Cherry_MX_1.00u_PCB"
+		(property "Footprint" "Macropad_Library:SW_Cherry_MX_1.00u_PCB"
 			(at 99.06 97.155 0)
 			(effects
@@
 			)
 		)
-		(property "Footprint" "Button_Switch_Keyboard:SW_Cherry_MX_1.00u_PCB"
+		(property "Footprint" "Macropad_Library:SW_Cherry_MX_1.00u_PCB"
 			(at 110.49 71.755 0)
 			(effects
@@
 			)
 		)
-		(property "Footprint" "Connector_PinHeader_2.54mm:PinHeader_1x04_P2.54mm_Vertical"
+		(property "Footprint" "Macropad_Library:SSD1306"
 			(at 235.458 82.55 0)
 			(effects
@@
 			)
 		)
-		(property "Footprint" "Button_Switch_Keyboard:SW_Cherry_MX_1.00u_PCB"
+		(property "Footprint" "Macropad_Library:SW_Cherry_MX_1.00u_PCB"
 			(at 110.49 47.625 0)
 			(effects
@@
 			)
 		)
-		(property "Footprint" "Button_Switch_THT:SW_PUSH-12mm"
+		(property "Footprint" "Macropad_Library:SW_PUSH-12mm"
 			(at 149.86 36.83 0)
 			(effects
@@
 			)
 		)
-		(property "Footprint" "Button_Switch_Keyboard:SW_Cherry_MX_1.00u_PCB"
+		(property "Footprint" "Macropad_Library:SW_Cherry_MX_1.00u_PCB"
 			(at 104.14 145.415 0)
 			(effects
@@
 			)
 		)
-		(property "Footprint" "Button_Switch_Keyboard:SW_Cherry_MX_1.00u_PCB"
+		(property "Footprint" "Macropad_Library:SW_Cherry_MX_1.00u_PCB"
 			(at 99.06 108.585 0)
 			(effects

Commit message: updated
Parts:
- SW1, SW2, SW3, SW4, SW5, SW6, SW7, SW8, SW9: value CherryMX -> Kailh Choc; footprint Macropad_Library:SW_Cherry_MX_1.00u_PCB -> Macropad_Library:SW_PG1350
- U2: footprint skqucaa010_joystick:SKQUCAA010 -> Macropad_Library:SKQUCAA010
Changed lines of the file:
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@@
 			)
 		)
-		(property "Value" "CherryMX"
+		(property "Value" "Kailh Choc"
 			(at 99.06 90.17 0)
 			(effects
@@
 			)
 		)
-		(property "Footprint" "Macropad_Library:SW_Cherry_MX_1.00u_PCB"
+		(property "Footprint" "Macropad_Library:SW_PG1350"
 			(at 99.06 85.725 0)
 			(effects
@@
 			)
 		)
-		(property "Value" "CherryMX"
+		(property "Value" "Kailh Choc"
 			(at 104.14 125.73 0)
 			(effects
@@
 			)
 		)
-		(property "Footprint" "Macropad_Library:SW_Cherry_MX_1.00u_PCB"
+		(property "Footprint" "Macropad_Library:SW_PG1350"
 			(at 104.14 121.285 0)
 			(effects
@@
 			)
 		)
-		(property "Value" "CherryMX"
+		(property "Value" "Kailh Choc"
 			(at 104.14 137.16 0)
 			(effects
@@
 			)
 		)
-		(property "Footprint" "Macropad_Library:SW_Cherry_MX_1.00u_PCB"
+		(property "Footprint" "Macropad_Library:SW_PG1350"
 			(at 104.14 132.715 0)
 			(effects
@@
 			)
 		)
-		(property "Value" "CherryMX"
+		(property "Value" "Kailh Choc"
 			(at 110.49 64.77 0)
 			(effects
@@
 			)
 		)
-		(property "Footprint" "Macropad_Library:SW_Cherry_MX_1.00u_PCB"
+		(property "Footprint" "Macropad_Library:SW_PG1350"
 			(at 110.49 60.325 0)
 			(effects
@@
 			)
 		)
-		(property "Value" "CherryMX"
+		(property "Value" "Kailh Choc"
 			(at 99.06 101.6 0)
 			(effects
@@
 			)
 		)
-		(property "Footprint" "Macropad_Library:SW_Cherry_MX_1.00u_PCB"
+		(property "Footprint" "Macropad_Library:SW_PG1350 "
 			(at 99.06 97.155 0)
 			(effects
@@
 			)
 		)
-		(property "Value" "CherryMX"
+		(property "Value" "Kailh Choc"
 			(at 110.49 76.2 0)
 			(effects
@@
 			)
 		)
-		(property "Footprint" "Macropad_Library:SW_Cherry_MX_1.00u_PCB"
+		(property "Footprint" "Macropad_Library:SW_PG1350"
 			(at 110.49 71.755 0)
 			(effects
@@
 		)
 		(property "Footprint" "Macropad_Library:SSD1306"
-			(at 235.458 82.55 0)
+			(at 215.392 81.28 0)
 			(effects
 				(font
@@
 			)
 		)
-		(property "Value" "CherryMX"
+		(property "Value" "Kailh Choc"
 			(at 110.49 52.07 0)
 			(effects
@@
 			)
 		)
-		(property "Footprint" "Macropad_Library:SW_Cherry_MX_1.00u_PCB"
+		(property "Footprint" "Macropad_Library:SW_PG1350"
 			(at 110.49 47.625 0)
 			(effects
@@
 			)
 		)
-		(property "Footprint" "skqucaa010_joystick:SKQUCAA010"
+		(property "Footprint" "Macropad_Library:SKQUCAA010"
 			(at 203.2 102.87 0)
 			(effects
@@
 			)
 		)
-		(property "Value" "CherryMX"
+		(property "Value" "Kailh Choc"
 			(at 104.14 149.86 0)
 			(effects
@@
 			)
 		)
-		(property "Footprint" "Macropad_Library:SW_Cherry_MX_1.00u_PCB"
+		(property "Footprint" "Macropad_Library:SW_PG1350"
 			(at 104.14 145.415 0)
 			(effects
@@
 			)
 		)
-		(property "Value" "CherryMX"
+		(property "Value" "Kailh Choc"
 			(at 99.06 113.03 0)
 			(effects
@@
 			)
 		)
-		(property "Footprint" "Macropad_Library:SW_Cherry_MX_1.00u_PCB"
+		(property "Footprint" "Macropad_Library:SW_PG1350"
 			(at 99.06 108.585 0)
 			(effects
